File: main_board.sch (KiCad schematic (older format))
At the start: 30 parts, among them P1 PIC_PROG, P4 CONN_2, P5 CONN_2, P6 CONN_4X2, P7 CONN_2, P8 CONN_2, P9 CONN_2, U1 PIC24EP256GP204, U2 MY_CONN_14X2, U4 BT_CONN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

Commit message: checking DFM of the layout
Parts:
- added R15: 1M, symbol R
- R1, R3, R5, R6, R7: value R -> 1K
- R10, R11, R12, R13, R14: value R -> 10K
- gave numbers to parts that had none: 3
- renumbered D3 to D2, D5 to D3, D6 to D4, D7 to D5
Connections:
- wire segments 97 -> 98
Other:
- moved on the sheet: CR1

Commit message: long time coming update
Parts:
- removed P6: CONN_4X2, symbol CONN_4X2
- removed U2: MY_CONN_14X2, symbol MY_CONN_14X2
- removed U4: BT_CONN, symbol BT_CONN
- removed U5: WOS_CONN, symbol WOS_CONN
- added C10, C9: 0.1uF, symbol C
- added D6: LED, symbol LED
- added R16, R20, R21: 10K, symbol R
- added R17: DNI, symbol R
- added R18: 330, symbol R
- added R22: 1K, symbol R
- added SW1: SPST, symbol SPST
- added U2: RN42DS, symbol RN42DS
- added U4: 2SD1757K, symbol 2SD1757K
Connections:
- net labels added: B1, B2, B3, B4, B5
- net labels removed: EE_nCS, I2C_CLK, I2C_DATA, INT1, INT2, JP3, MRF_nCS, SCK1, SDI1, SDO1, SPI_CLK, SPI_DIN, SPI_DOUT, UART1_RX, UART1_TX, WAKE, nRESET
- wire segments 98 -> 71
- no-connect marks 22 -> 37
Other:
- note removed: "Bluetooth Connection"
- note removed: "I2C Connection"
- note removed: "Microchip\nWireless"
- note removed: "Wake on Shake Connection"
- moved on the sheet: R10, R11, R12, R13, R14
