File: pic24_power.sch (KiCad schematic (older format))
At the start: 12 parts, among them P2 BAT_CONN, P3 PWR_SWITCH, U1 PIC24EP256GP204, U3 TLV1117

Commit message: checking DFM of the layout
Parts:
- added C6, C7: 0.1uF, symbol C
- C1, C2, C4: value C -> 10uF
- C3, C5: value C -> 0.1uF
- R9: value R -> 1K
Connections:
- net GND: now also C6.2, C7.2
- net VDD: now also R9.2, C6.1, C7.1; no longer R9.1
- net at D8.1 (A): now also R9.1; no longer R9.2
Other:
- moved on the sheet: C1, C2, C3, C4, C5, D8, P2, P3, R8, R9, U1B, U3

Commit message: long time coming update
Parts:
- removed P3: PWR_SWITCH, symbol PWR_SWITCH
- removed U3: TLV1117, symbol TLV1117
- added C8: 0.1uF, symbol C
- added P3: CONN_2, symbol CONN_2
- added P6: BAT_CONN, symbol BAT_CONN
- added TP1, TP2: TEST_POINT, symbol TEST_POINT
- added U3: TPS73633MDBVREP, symbol TPS73633MDBVREP
- C4: value 10uF -> 0.1uF
- renumbered D8 to D7
Connections:
- net +BATT: now also P3.2 (PM), U3.1 (IN), U3.3 (EN)
- net GND: now also U1.16 (AVSS), C8.2, P6.2 (VSS), TP1.1, TP2.1, U3.2 (GND); no longer U1.17 (AVDD)
- net VDD: now also U3.5 (OUT)
- net at P2.1 (VDD): now also P3.1 (P1), P6.1 (VDD)
- net at R8.2: now also U1.17 (AVDD); no longer U1.16 (AVSS)
- new net: C8.1, U3.4 (NR)
- no-connect marks 1 -> 0
Other:
- note added: "Mounting holes"
- moved on the sheet: P2, R8
